File: Joystick-Controller-PCB/Joystick-Controller.kicad_pcb (KiCad board)
At the start: 2 copper layers, 214.5 x 91.5 mm, 22 parts, among them J1 Conn_01x28_Socket, J2 Conn_01x28_Socket, J3 Conn_01x03_Socket, J4 Conn_01x04_Socket, J5 TFT_Display_Conn_Socket, J6 TFT_SD_Conn_Socket, SW1 COM-10302, SW3 COM-10302

Commit message: Iteration 1
Routing:
- net VBUS: track 17.8 -> 184.3 mm
- net /GPIO40_ADC0: track 0.00 -> 115.0 mm
- net /GPIO41_ADC1: track 0.00 -> 111.6 mm
- net /GPIO20: track 0.00 -> 77.1 mm
- net /GPIO38: track 7.85 -> 82.5 mm, vias 0 -> 1
- net /GPIO39: track 8.51 -> 53.3 mm
- net /GPIO30: track 0.00 -> 24.7 mm, vias 0 -> 1
- net /GPIO29: track 0.00 -> 22.5 mm
- net /GPIO31: track 0.00 -> 21.5 mm
- net GND: track 76.2 -> 87.3 mm, vias 0 -> 1
- net /GPIO0: track 94.4 -> 91.3 mm

Commit message: pcb files checked by Niraj
Parts:
- moved J1 0.75 mm to (205.7, 58.4)
- moved J2 0.75 mm to (205.7, 76.2)
- moved J3 0.75 mm to (119.4, 58.4)
- moved J4 0.74 mm to (121.9, 76.2)
Changed lines of the file:
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@@
 	(footprint "Connector_PinSocket_2.54mm:PinSocket_1x28_P2.54mm_Vertical"
 		(layer "F.Cu")
-		(at 206.36 75.78 -90)
+		(at 205.74 76.2 -90)
 		(descr "Through hole straight socket strip, 1x28, 2.54mm pitch, single row (from Kicad 4.0.7), script generated")
 		(tags "Through hole socket strip THT 1x28 2.54mm single row")
@@
 	(footprint "Connector_PinSocket_2.54mm:PinSocket_1x04_P2.54mm_Vertical"
 		(layer "F.Cu")
-		(at 122.543093 75.79672 -90)
+		(at 121.92 76.2 -90)
 		(descr "Through hole straight socket strip, 1x04, 2.54mm pitch, single row (from Kicad 4.0.7), script generated")
 		(tags "Through hole socket strip THT 1x04 2.54mm single row")
@@
 	(footprint "Connector_PinSocket_2.54mm:PinSocket_1x28_P2.54mm_Vertical"
 		(layer "F.Cu")
-		(at 206.36 58 -90)
+		(at 205.74 58.42 -90)
 		(descr "Through hole straight socket strip, 1x28, 2.54mm pitch, single row (from Kicad 4.0.7), script generated")
 		(tags "Through hole socket strip THT 1x28 2.54mm single row")
@@
 	(footprint "Connector_PinSocket_2.54mm:PinSocket_1x03_P2.54mm_Vertical"
 		(layer "F.Cu")
-		(at 120 58 -90)
+		(at 119.38 58.42 -90)
 		(descr "Through hole straight socket strip, 1x03, 2.54mm pitch, single row (from Kicad 4.0.7), script generated")
 		(tags "Through hole socket strip THT 1x03 2.54mm single row")
@@
 		)
 	)
-	(group ""
-		(members "00673a4f-801a-40e1-8442-1fa9b305b949" "11708747-462e-48b6-9c69-d159efe21a26"
-			"6e23b6a5-80f1-4689-b8fa-a8cdf4fa0723" "d8837136-f24e-42a9-bc77-9d0b16ca4ff8"
-		)
-	)

Commit message: Board Complete
Parts:
- removed SW1, SW3: COM-10302, footprints:COM-10302_SPK
- added S1: SW_B3F-4055, B3F_4055:SW_B3F-4055, F.Cu at (225.8, 88.5)
- added S2: SW_B3F-4055, B3F_4055:SW_B3F-4055, F.Cu at (250.2, 88.5)
- D1: value POWER LED -> PWR
- D3: value USER LED -> USER
- R1, R7: value 1000 -> 10k
- R2, R3, R4, R5, R6: value 220 -> 100
Routing:
- net /GPIO38: track 82.5 -> 85.1 mm
- net /GPIO41_ADC1: track 111.6 -> 113.7 mm
- net /GPIO39: track 53.3 -> 54.6 mm
- net /GPIO20: track 77.1 -> 78.3 mm
- net /GPIO40_ADC0: track 115.0 -> 116.0 mm
- net /SWD: track 28.7 -> 29.2 mm
- net /GPIO0: track 91.3 -> 91.9 mm
Other:
- board text added: "Color"
- board text added: "Roy, Andrew, Bryan, Jackie"
- board text added: "Save"

Commit message: Updated LED part and resistor values. Added footprint for switch and RGB LED
Parts:
- removed D2: COLOR INDICATOR, LED_SMD:LED_RGB_5050-6
- added LED1: ~, ProLib_pcs_2025-11-13:LED-SMD_6PIN-L1.60-W1.50-BL-RD, F.Cu at (228.2, 49.8)
- D1: value PWR -> POWER LED
- D3: value USER -> USER LED
- R3, R5: value 100 -> 10
- R4: value 100 -> 68
- S1, S2: value SW_B3F-4055 -> B3F-4055
- moved R3 8.00 mm to (215.5, 52.5)
- moved R5 8.00 mm to (215.5, 44.5)
Connections:
- R3 pad 2: /GPIO5 -> /GPIO3
- R5 pad 2: /GPIO3 -> /GPIO5
- S1 pad 2: (no net) -> +3V3
- S1 pad 4: (no net) -> /GPIO39
- S2 pad 2: (no net) -> +3V3
- S2 pad 4: (no net) -> /GPIO38
Routing:
- net Net-(LED1---Pad2): track 25.4 -> 11.9 mm
- net /GPIO38: track 85.1 -> 97.6 mm
- net /GPIO39: track 54.6 -> 67.1 mm
- net Net-(LED1---Pad6): track 10.0 -> 13.7 mm
- net Net-(LED1---Pad4): track 14.8 -> 11.6 mm
- net /GPIO5: track 31.5 -> 32.3 mm
- net /GPIO3: track 23.1 -> 23.9 mm
